Commit message: Added marching cubes for bucket

File: excavator-visualizer/urdf/electrical_excavator.urdf.xacro (robot description, xacro)
@@ -4,4 +4,11 @@
   <xacro:include filename="_materials.urdf.xacro" />
   <link name="world" />
+  <link name="container" />
+  <joint name="Container" type="fixed">
+    <axis xyz="0.0 0.0 1.0" />
+    <origin xyz="0.0 -2.0 -0.75" rpy="0 0 0" />
+    <parent link="world"/>
+    <child link="container"/>
+  </joint>
   <link name="base">
     <visual>

Commit message: updated

File: excavator-visualizer/urdf/electrical_excavator.urdf.xacro (robot description, xacro)
@@ -5,4 +5,11 @@
   <link name="world" />
   <link name="container" />
+  <link name="map" />
+  <joint name="camera" type="fixed">
+     <axis xyz="0.0 0.0 1.0" />
+    <origin xyz="0.0 0.0 1.0" rpy="0 0 0" />
+    <parent link="world"/>
+    <child link="map"/>
+  </joint>
   <joint name="Container" type="fixed">
     <axis xyz="0.0 0.0 1.0" />
